File: baseboard/cad/1590N1 IO Board.kicad_pcb (KiCad board)
At the start: 4 copper layers, 58 x 77 mm, 96 parts, among them J1 DC POWER JACK, J12 6-440054-2, J13 6-440054-2, J16 Conn_01x04_Pin, J17 6-440054-2, J18 6-440054-2, J2 1/4" JACK, STEREO, J23 2P_HEADER, J24 2P_HEADER, J25 2P_HEADER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

Commit message: finished initial layout
Parts:
- added REF**: OSHW-Logo_5.7x6mm_SilkScreen, Symbol:OSHW-Logo_5.7x6mm_SilkScreen, F.Cu at (141.4, 141.6)
- added REF**: ESD-Logo_6.6x6mm_SilkScreen, Symbol:ESD-Logo_6.6x6mm_SilkScreen, F.Cu at (134.5, 141.7)
- G1, G2, G3: moved to B.Cu
- U1: footprint Package_DFN_QFN:QFN-32-1EP_5x5mm_P0.5mm_EP3.45x3.45mm_ThermalVias -> Library:QFN-32-1EP_5x5mm_P0.5mm_EP3.45x3.45mm_ThermalVias
- U3: footprint Package_CSP:LFCSP-20-1EP_4x4mm_P0.5mm_EP2.6x2.6mm -> Library:LFCSP-20-1EP_4x4mm_P0.5mm_EP2.6x2.6mm
- U8: footprint Package_DFN_QFN:DFN-10-1EP_3x3mm_P0.5mm_EP1.65x2.38mm_ThermalVias -> Library:DFN-10-1EP_3x3mm_P0.5mm_EP1.65x2.38mm_ThermalVias
- moved C26 122.3 mm to (105.2, 111.0), turned to 90 degrees
- moved C15 101.7 mm to (131.6, 132.1), turned to 180 degrees
- moved Q1 97.8 mm to (108.5, 137.7), turned to 180 degrees
- moved C20 93.7 mm to (149.7, 135.4), turned to 180 degrees
- moved L2 93.5 mm to (137.6, 129.3), turned to 180 degrees
- moved C11 93.5 mm to (135.0, 129.3), turned to 90 degrees
- moved R21 93.2 mm to (105.1, 138.0), turned to -90 degrees
- moved C28 92.5 mm to (119.5, 138.0), turned to 90 degrees
- moved C14 92.4 mm to (144.8, 132.6), turned to 90 degrees
- moved L1 92.3 mm to (140.6, 129.3), turned to 180 degrees
- moved D9 90.0 mm to (102.1, 119.0), turned to 180 degrees
- moved C10 89.9 mm to (139.1, 126.1), turned to -90 degrees
- moved R6 89.3 mm to (136.6, 135.7), turned to 90 degrees
- moved R18 88.7 mm to (117.5, 137.9), turned to -90 degrees
- moved R20 88.6 mm to (111.8, 138.0), turned to -90 degrees
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- renumbered U9 to U4
Connections:
- U1 pad 17: unconnected-(U1-PB2-Pad17) -> V_FTSW_B
- U1 pad 18: unconnected-(U1-PA8-Pad18) -> V_FTSW_A
- U1 pad 19: unconnected-(U1-PA9/NC-Pad19) -> +12V_EN
- U1 pad 20: unconnected-(U1-PC6-Pad20) -> -12V_EN
- U1 pad 21: +12V_EN -> unconnected-(U1-PA10/NC-Pad21)
- U1 pad 22: -12V_EN -> unconnected-(U1-PA11/PA9-Pad22)
- U1 pad 23: V_FTSW_B -> unconnected-(U1-PA12/PA10-Pad23)
- U1 pad 24: V_FTSW_A -> unconnected-(U1-PA13-Pad24)
- U1 pad 28: VLED2 -> unconnected-(U1-PB4-Pad28)
- U1 pad 29: VLED1 -> unconnected-(U1-PB5-Pad29)
- U1 pad 8: unconnected-(U1-PA1-Pad8) -> VLED2
- U1 pad 9: unconnected-(U1-PA2-Pad9) -> VLED1
Routing:
- net +9V: track 9.79 -> 102.6 mm, vias 2 -> 4
- net +3V3: track 2.34 -> 91.0 mm, vias 1 -> 3
- net GND: track 51.6 -> 102.3 mm, vias 19 -> 54
- net -9V: track 12.1 -> 52.9 mm, vias 2 -> 4
- net +12V_EN: track 0.00 -> 35.3 mm, vias 0 -> 2
- net -12V_EN: track 0.00 -> 34.7 mm, vias 0 -> 2
- net AUDIO_IN_A: track 0.00 -> 27.2 mm, vias 0 -> 1
- net AUDIO_IN_B: track 0.00 -> 27.0 mm
- net AUDIO_OUT_B: track 0.00 -> 25.8 mm, vias 0 -> 1
- net AUDIO_OUT_A: track 0.00 -> 24.7 mm
- net DC_IN: track 38.2 -> 57.4 mm, vias 2 -> 6
- net -Vsw: track 0.00 -> 16.4 mm, vias 0 -> 2
- net SWDCK: track 0.00 -> 13.9 mm
- net SWDIO: track 0.00 -> 11.2 mm
- net V_FTSW_B: track 0.00 -> 10.4 mm
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- added copper zone on F.Cu, net +9V
- added copper zone on F.Cu, net +Vsw
- added copper zone on F.Cu, net -9V
- added copper zone on B.Cu, net -Vsw
- added copper zone on F.Cu, net -Vsw
- added copper zone on F.Cu, net /Power/FB1
- added copper zone on F.Cu, net /Power/FB2
- added copper zone on F.Cu, net /Power/VSW1
- added copper zone on F.Cu, net /Power/VSW2
- added copper zone on F.Cu, net /Power/V_SW_D2
- added copper zone on F.Cu, net Net-(U8-VREF)
Other:
- board text added: "AIR Baseboard V0.9"
- board text added: "RST"
- board text added: "⎓"
- board text added: "⏚"
