File: hardware/cad/1590N1 IO Board.kicad_pcb (KiCad board)
At the start: 4 copper layers, 58 x 77 mm, 117 parts, among them J1 1/4" JACK, STEREO, J11 6-440054-2, J12 6-440054-2, J15 Conn_01x20_Pin, J16 Conn_01x20_Pin, J2 DC POWER JACK, J3 6-440054-2, J5 1/4" JACK, STEREO, J6 Conn_01x04_Pin, J7 6-440054-2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

Commit message: more layout updates
Parts:
- removed the C24 at (54.2, 110.3)
- removed the C25 at (136.0, 78.9)
- removed C48, C49, C50: 22μF, Capacitor_SMD:C_0805_2012Metric
- added C28: 10n, Capacitor_SMD:C_0603_1608Metric, F.Cu at (181.5, 83.4)
- added C29: 10n, Capacitor_SMD:C_0603_1608Metric, F.Cu at (181.5, 85.9)
- added G1: Chassis, Library:Harwin_EMI_Finger_S7061-46R, F.Cu at (181.7, 115.4)
- C1, C15: value 6pF -> 6p
- C10, C11, C12, C13, C2, C3, C4, C5, C6, C7, C8, C9: value 330nF -> 330n
- C14, C16, C17, C18, C19, C20, C21, C22, C23: value 22μF -> 22u
- C24: renamed from C26; value 100nF -> 100n
- C25: renamed from C27; value 100nF -> 100n
- C26: renamed from C28; value 100nF -> 100n
- C27: renamed from C29; value 100nF -> 100n
- C30, C37, C38: value 10nF -> 100n
- C31: value 10nF -> 22u; footprint Capacitor_SMD:C_0603_1608Metric -> Capacitor_SMD:C_0805_2012Metric
- C32, C41: value 100nF -> 22u; footprint Capacitor_SMD:C_0603_1608Metric -> Capacitor_SMD:C_0805_2012Metric
- C33, C34, C44: value 22μF -> 100n
- C35, C36: value 100nF -> 10n; footprint Capacitor_SMD:C_0805_2012Metric -> Capacitor_SMD:C_0603_1608Metric
- C39, C43: value 100nF -> 100n
- C40, C42: value 100nF -> 100n; footprint Capacitor_SMD:C_0603_1608Metric -> Capacitor_SMD:C_0805_2012Metric
- C45, C46, C47: value 100nF -> 22u
- L1: value 11µH -> 11u
- L2, L3: value 15μH -> 15u
- R1, R2: value 1MΩ -> 1M
- R10, R11, R13, R7: value 62kΩ -> 62k
- R12, R14, R17, R9: value 499kΩ -> 499k
- R15, R16: value 78.7kΩ -> 78.7k
- R18, R19, R20, R21, R22, R23, R24, R5, R6: value 49.9KΩ -> 49.9K
- R25, R27, R28, R29: value 47Ω -> 47R
- R26, R30, R8: value 10kΩ -> 10k
- R3, R4: value 0Ω -> 0R
- U3, U4: value REF** -> OPA1679
- U8: footprint Package_CSP:LFCSP-20-1EP_4x4mm_P0.5mm_EP2.6x2.6mm -> Package_CSP:LFCSP-20-1EP_4x4mm_P0.5mm_EP2.6x2.6mm_ThermalVias
- moved C38 73.1 mm to (90.2, 131.4), turned to 90 degrees
- moved C20 66.6 mm to (198.2, 83.6)
- moved C21 66.6 mm to (198.2, 86.7)
- moved C22 66.6 mm to (198.2, 89.7)
- moved U2 66.3 mm to (198.2, 96.5)
- moved C23 65.2 mm to (198.2, 92.7)
- moved C33 64.4 mm to (202.6, 89.7)
- moved C34 64.4 mm to (202.6, 92.7)
- moved C16 63.1 mm to (193.7, 83.6)
- moved C17 63.1 mm to (193.7, 86.7)
- moved C18 63.1 mm to (193.7, 89.7)
- moved C19 63.1 mm to (193.7, 92.7)
- moved U5 61.3 mm to (198.1, 101.2)
- moved C26 59.7 mm to (81.1, 111.6), turned to 90 degrees
- moved C32 58.6 mm to (202.6, 86.7)
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- renumbered G1 to G2, G2 to G3
Connections:
- C24 pad 2: Net-(U3E-V+) -> +9V
- C25 pad 1: Net-(U3E-V-) -> -9V
- C26 pad 2: Net-(U4E-V+) -> +9V
- C27 pad 1: Net-(U4E-V-) -> -9V
- C30 pad 1: +9V -> GND
- C30 pad 2: Net-(U5-BYPP) -> +3V3
- C31 pad 1: -9V -> GND
- C31 pad 2: /Power/VBYPN -> +9V
- C32 pad 1: GND -> -9V
- C32 pad 2: +3V3 -> GND
- C35 pad 1: GND -> +9V
- C35 pad 2: +9V -> GND
- C36 pad 1: -9V -> GND
- C36 pad 2: GND -> -9V
- C37 pad 1: +9V -> GND
- C37 pad 2: GND -> +3V3
- C38 pad 2: -9V -> +9V
- C39 pad 1: GND -> -9V
- C39 pad 2: +3V3 -> GND
- C40 pad 2: +9V -> +3V3
- C41 pad 1: -9V -> GND
- C41 pad 2: GND -> Net-(C41-Pad2)
- C42 pad 1: -9V -> GND
- C42 pad 2: +9V -> +3V3
- C44 pad 2: Net-(C44-Pad2) -> +3V3
- C45 pad 2: +3V3 -> Net-(C45-Pad2)
- C46 pad 2: +3V3 -> +9V
- C47 pad 2: +3V3 -> -9V
- CHS1 pad 1: PWR -> GND
- CHS2 pad 1: PWR -> GND
- R23 pad 1: Net-(U4B--B) -> Net-(U4C--C)
- R23 pad 2: Net-(U4C--C) -> Net-(U4B--B)
- R24 pad 1: Net-(U4C--C) -> Net-(U4B--B)
- R24 pad 2: Net-(U4D-+D) -> Net-(U4A-+A)
- R25 pad 1: Net-(C44-Pad2) -> Net-(C41-Pad2)
- R26 pad 1: Net-(C44-Pad2) -> Net-(C41-Pad2)
- R29 pad 1: Net-(C48-Pad2) -> Net-(C45-Pad2)
- R30 pad 1: Net-(C48-Pad2) -> Net-(C45-Pad2)
- U3 pad 10: Net-(U3E-V-) -> -9V
- U3 pad 3: Net-(U3E-V+) -> +9V
- U4 pad 1: AUDIO_OUT_FILT+ -> AUDIO_OUT_FILT-
- U4 pad 10: Net-(U4E-V-) -> -9V
- U4 pad 11: Net-(U4D-+D) -> AUDIO_OUT_SE
- U4 pad 12: AUDIO_OUT_FILT- -> AUDIO_OUT_FILT+
- U4 pad 14: AUDIO_OUT_FILT- -> AUDIO_OUT_FILT+
- U4 pad 15: AUDIO_OUT_FILT+ -> AUDIO_OUT_FILT-
- U4 pad 2: AUDIO_OUT_SE -> Net-(U4A-+A)
- U4 pad 3: Net-(U4E-V+) -> +9V
- U4 pad 4: AUDIO_OUT_SE -> GND
- U4 pad 6: Net-(U4B--B) -> Net-(U4A-+A)
- U4 pad 7: Net-(U4D-+D) -> Net-(U4C--C)
- U4 pad 9: GND -> AUDIO_OUT_SE
- U5 pad 11: /Power/VBYPN -> Net-(U5-BYPN)
- U5 pad 3: Net-(U5-BYPP) -> /Power/VBYPP
- U6 pad 1: Net-(C44-Pad2) -> Net-(C41-Pad2)
- U6 pad 3: Net-(C48-Pad2) -> Net-(C45-Pad2)
Routing:
- net Net-(U4A-+A): track 0.00 -> 17.2 mm
- net AUDIO_OUT_SE: track 0.00 -> 12.6 mm
- net Net-(R20-Pad2): track 10.2 -> 2.85 mm
- net /Microcontroller and Switching/BYPASS_A: track 0.00 -> 7.23 mm, vias 0 -> 2
- net -9V: track 0.00 -> 7.20 mm, vias 0 -> 3
- net Net-(U3E-V+): track 6.97 -> 0.00 mm, vias 1 -> 0
- net Net-(U3A--A): track 18.5 -> 12.1 mm
- net GND: track 15.2 -> 21.3 mm, vias 4 -> 10
- net Net-(U3E-V-): track 5.25 -> 0.00 mm, vias 1 -> 0
- net /Microcontroller and Switching/AUDIO_A_TO_B: track 0.00 -> 4.67 mm, vias 0 -> 2
- net /Microcontroller and Switching/BYPASS_B: track 0.00 -> 4.57 mm, vias 0 -> 2
- net AUDIO_OUT_FILT+: track 4.70 -> 9.06 mm
- net AUDIO_OUT_FILT-: track 4.70 -> 9.06 mm
- net Net-(U3C--C): track 18.0 -> 21.3 mm
- net Net-(U4B--B): track 0.00 -> 3.24 mm
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- added copper zone on F.Cu, net +9V
- added copper zone on F.Cu, net -9V
- added copper zone on F.Cu, net GND
