File: hardware/cad/audio.kicad_sch (KiCad schematic)
At the start: 18 parts, among them J201 1/4" JACK, STEREO, J203 1/4" JACK, STEREO, J308 FFC CONNECTOR, U302 ADG5434

Commit message: finalized schematic
Parts:
- added FID303: FIDUCIAL, Fiducial:Fiducial_0.5mm_Mask1mm, symbol Mechanical:Fiducial
- C18, C38: value 100n -> 100nF
- C201, C210: value 150p -> 150pF
- C414: value 39n -> 39nF
- C418: value 2.2µ -> 2.2µF
- G2: value Chassis -> CHASSIS
- R201: value 1M -> 1MΩ
- R202: value 49.9k -> 49.9kΩ
Other:
- note added: "PLACE C201 AS CLOSE TO J201 AS POSSIBLE PLACE C210 AS CLOSE TO J203 AS POSSIBLE CAPACITORS C201, C202, C209, C210: 10% TOLERANCE, METALLIZED PET FILM DIELECTRIC PLACE CHASSIS GROUNDS AS CLOSE TO AUDIO JACKS AS POSSIBLE PLACE BYPASS CAPACITORS AS CLOSE TO ICS OR CONNECTORS AS POSSIBLE PLACE CONNECTORS NEAR BOARD EDGE PLACE AUDIO COMPONENTS NEAR EACH OTHER AND AWAY FROM OTHER CIRCUITS"
- note removed: "PLACE C201 AS CLOSE TO J201 AS POSSIBLE PLACE C210 AS CLOSE TO J203 AS POSSIBLE CAPACITORS C201, C202, C209, C210: 10% TOLERANCE, METALLIZED PET FILM DIELECTRIC PLACE CHASSIS GROUNDs AS CLOSE TO AUDIO JACKS AS POSSIBLE PLACE BYPASS CAPACITORS AS CLOSE TO IC OR CONNECTOR AS POSSIBLE PLACE CONNECTORS NEAR BOARD EDGE"
- company: Alessandro Rizzoni -> ALESSANDRO RIZZONI
- title: Baseboard -> BASEBOARD
Changed lines of the file:
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@@
   (paper "USLedger")
   (title_block
-    (title "Baseboard")
+    (title "BASEBOARD")
     (date "2023-04-28")
     (rev "A")
-    (company "Alessandro Rizzoni")
+    (company "ALESSANDRO RIZZONI")
     (comment 1 "SCHEMATIC")
     (comment 2 "DRAFT")
@@
     (effects (font (size 1.27 1.27) (thickness 0.254) bold) (justify left bottom))
   )
-  (text "PLACE C201 AS CLOSE TO J201 AS POSSIBLE\nPLACE C210 AS CLOSE TO J203 AS POSSIBLE\nCAPACITORS C201, C202, C209, C210: 10% TOLERANCE, METALLIZED PET FILM DIELECTRIC\nPLACE CHASSIS GROUNDs AS CLOSE TO AUDIO JACKS AS POSSIBLE\nPLACE BYPASS CAPACITORS AS CLOSE TO IC OR CONNECTOR AS POSSIBLE\nPLACE CONNECTORS NEAR BOARD EDGE"
+  (text "PLACE C201 AS CLOSE TO J201 AS POSSIBLE\nPLACE C210 AS CLOSE TO J203 AS POSSIBLE\nCAPACITORS C201, C202, C209, C210: 10% TOLERANCE, METALLIZED PET FILM DIELECTRIC\nPLACE CHASSIS GROUNDS AS CLOSE TO AUDIO JACKS AS POSSIBLE\nPLACE BYPASS CAPACITORS AS CLOSE TO ICS OR CONNECTORS AS POSSIBLE\nPLACE CONNECTORS NEAR BOARD EDGE\nPLACE AUDIO COMPONENTS NEAR EACH OTHER AND AWAY FROM OTHER CIRCUITS\n"
     (at 16.51 262.89 0)
     (effects (font (size 1.27 1.27)) (justify left bottom))
@@
     )
   )
+  (symbol (lib_id "Mechanical:Fiducial") (at 88.9 165.1 0) (unit 1)
+    (in_bom yes) (on_board yes) (dnp no) (fields_autoplaced)
+    (property "Reference" "FID303" (at 91.44 163.83 0)
+      (effects (font (size 1.27 1.27)) (justify left))
+    )
+    (property "Value" "FIDUCIAL" (at 91.44 166.37 0)
+      (effects (font (size 1.27 1.27)) (justify left))
+    )
+    (property "Footprint" "Fiducial:Fiducial_0.5mm_Mask1mm" (at 88.9 165.1 0)
+      (effects (font (size 1.27 1.27)) hide)
+    )
+    (property "Datasheet" "N/A" (at 88.9 165.1 0)
+      (effects (font (size 1.27 1.27)) hide)
+    )
+    (property "Manufacturer" "N/A" (at 88.9 165.1 0)
+      (effects (font (size 1.27 1.27)) hide)
+    )
+    (property "Part Number" "N/A" (at 88.9 165.1 0)
+      (effects (font (size 1.27 1.27)) hide)
+    )
+    (instances
+      (project "baseboard"
+        (path "/190888c1-6ce2-4681-a836-dc477e444e49/229a97b2-4425-47f7-b588-f32dc6b9bc79"
+          (reference "FID303") (unit 1)
+        )
+        (path "/190888c1-6ce2-4681-a836-dc477e444e49"
+          (reference "FID103") (unit 1)
+        )
+        (path "/190888c1-6ce2-4681-a836-dc477e444e49/e436358c-d730-4540-92b5-b7475a7c4a63"
+          (reference "FID201") (unit 1)
+        )
+      )
+    )
+  )
   (symbol (lib_id "power:-9V") (at 279.4 190.5 0) (mirror y) (unit 1)
     (in_bom yes) (on_board yes) (dnp no)
@@
       (effects (font (size 1.27 1.27)))
     )
-    (property "Value" "39n" (at 139.7 83.82 90)
+    (property "Value" "39nF" (at 139.7 83.82 90)
       (effects (font (size 1.27 1.27)))
     )
@@
       (effects (font (size 1.27 1.27)) (justify left))
     )
-    (property "Value" "100n" (at 275.59 203.2 0)
+    (property "Value" "100nF" (at 275.59 203.2 0)
       (effects (font (size 1.27 1.27)) (justify left))
     )
@@
       (effects (font (size 1.27 1.27)) hide)
     )
-    (property "Value" "Chassis" (at 336.55 91.44 0)
+    (property "Value" "CHASSIS" (at 336.55 91.44 0)
       (effects (font (size 1.27 1.27)))
     )
@@
       (effects (font (size 1.27 1.27)) (justify left))
     )
-    (property "Value" "2.2µ" (at 270.51 193.04 0)
+    (property "Value" "2.2µF" (at 270.51 193.04 0)
       (effects (font (size 1.27 1.27)) (justify left))
     )
@@
       (effects (font (size 1.27 1.27)) (justify left))
     )
-    (property "Value" "150p" (at 116.84 82.55 0)
+    (property "Value" "150pF" (at 116.84 82.55 0)
       (effects (font (size 1.27 1.27)) (justify left))
     )
@@
       (effects (font (size 1.27 1.27)) (justify right))
     )
-    (property "Value" "49.9k" (at 320.04 83.82 0)
+    (property "Value" "49.9kΩ" (at 320.04 83.82 0)
       (effects (font (size 1.27 1.27)) (justify right))
     )
@@
       (effects (font (size 1.27 1.27)) (justify left))
     )
-    (property "Value" "1M" (at 129.54 83.82 0)
+    (property "Value" "1MΩ" (at 129.54 83.82 0)
       (effects (font (size 1.27 1.27)) (justify left))
     )
@@
       (effects (font (size 1.27 1.27)))
     )
-    (property "Value" "39n" (at 304.8 71.12 90)
+    (property "Value" "39nF" (at 304.8 71.12 90)
       (effects (font (size 1.27 1.27)))
     )
@@
       (effects (font (size 1.27 1.27)) (justify left))
     )
-    (property "Value" "100n" (at 149.86 179.07 0)
+    (property "Value" "100nF" (at 149.86 179.07 0)
       (effects (font (size 1.27 1.27)) (justify left))
     )
@@
       (effects (font (size 1.27 1.27)) (justify left))
     )
-    (property "Value" "100n" (at 149.86 217.17 0)
+    (property "Value" "100nF" (at 149.86 217.17 0)
       (effects (font (size 1.27 1.27)) (justify left))
     )
@@
       (effects (font (size 1.27 1.27)) (justify left))
     )
-    (property "Value" "2.2µ" (at 288.29 203.2 0)
+    (property "Value" "2.2µF" (at 288.29 203.2 0)
       (effects (font (size 1.27 1.27)) (justify left))
     )
@@
       (effects (font (size 1.27 1.27)) hide)
     )
-    (property "Value" "Chassis" (at 106.68 92.71 0)
+    (property "Value" "CHASSIS" (at 106.68 92.71 0)
       (effects (font (size 1.27 1.27)))
     )
@@
       (effects (font (size 1.27 1.27)) (justify left))
     )
-    (property "Value" "100n" (at 257.81 193.04 0)
+    (property "Value" "100nF" (at 257.81 193.04 0)
       (effects (font (size 1.27 1.27)) (justify left))
     )
@@
       (effects (font (size 1.27 1.27)) (justify left))
     )
-    (property "Value" "150p" (at 334.01 82.55 0)
-      (effects (font (size 1.27 1.27)) (justify left))
-    )
+    (property "Value" "150pF" (at 334.01 82.55 0)
+      (effects (font (size 1.27 1.27)) (justify left))
+    )

Commit message: board layout first pass
Parts:
- C418: value 2.2µF -> 2.2μF
- U302: footprint Library:LFCSP-20-1EP_4x4mm_P0.5mm_EP2.6x2.6mm -> Library:LFCSP-20-1EP_4x4mm_P0.5mm_EP2.6x2.6mm_ThermalVias
Changed lines of the file:
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@@
       (effects (font (size 1.27 1.27)) (justify left))
     )
-    (property "Value" "2.2µF" (at 270.51 193.04 0)
+    (property "Value" "2.2μF" (at 270.51 193.04 0)
       (effects (font (size 1.27 1.27)) (justify left))
     )
@@
       (effects (font (size 1.27 1.27)) (justify left))
     )
-    (property "Value" "2.2µF" (at 288.29 203.2 0)
+    (property "Value" "2.2μF" (at 288.29 203.2 0)
       (effects (font (size 1.27 1.27)) (justify left))
     )
@@
       (effects (font (size 1.27 1.27)) (justify left))
     )
-    (property "Footprint" "Library:LFCSP-20-1EP_4x4mm_P0.5mm_EP2.6x2.6mm" (at 104.14 168.91 0)
+    (property "Footprint" "Library:LFCSP-20-1EP_4x4mm_P0.5mm_EP2.6x2.6mm_ThermalVias" (at 104.14 168.91 0)
       (effects (font (size 1.27 1.27)) (justify left) hide)
     )

Commit message: an inappropriately large commit
Parts:
- removed C18 (x2): 100nF, Capacitor_SMD:C_0402_1005Metric, symbol Device:C
- removed FID303: FIDUCIAL, Fiducial:Fiducial_0.5mm_Mask1mm, symbol Mechanical:Fiducial
- removed U302: ADG5434, Library:LFCSP-20-1EP_4x4mm_P0.5mm_EP2.6x2.6mm_ThermalVias, symbol Library:Analog_Devices_ADG5433
- added C18 (x2): 100nF, Capacitor_SMD:C_0402_1005Metric, symbol Device:C
- added U201: ADG5434, Library:LFCSP-20-1EP_4x4mm_P0.5mm_EP2.6x2.6mm, symbol Library:Analog_Devices_ADG5433
- C38: Part Number GRM155R61H104KE19J -> GRM188C71E225KE11D
- C414: footprint Capacitor_SMD:C_0603_1608Metric -> Capacitor_SMD:C_0805_2012Metric; Manufacturer Murata -> TDK; Part Number GCD188R71E393KA01 -> C2012C0G2A333J125AC
- C418: Part Number GRM188R61H225KE11J -> GRM188Z71E225KE43D
- J201, J203: value 1/4" JACK, STEREO -> ACJS-IHS
- J308: value FFC CONNECTOR -> SFV20R-2STE1HLF; symbol Connector_Generic_MountingPin:Conn_01x20_MountingPin -> Library:Conn_01x20_SHIELD
- R201: Part Number (none) -> RK73H1ETTP1004F
- R202: Part Number (none) -> RK73H1ETTP4992F
Connections:
- net +9V: now also C18.1, U201.13 (VDD)
- net -9V: now also C18.1, U201.21 (VSS), U201.3 (VSS)
- net AUDIO_A_TO_B: now also U201.11 (D3), U201.6 (D2)
- net AUDIO_IN_A: now also U201.1 (D1)
- net AUDIO_IN_B: now also U201.10 (S3A)
- net AUDIO_IN_FILT: now also U201.20 (S1A)
- net AUDIO_OUT_A: now also U201.5 (S2B)
- net AUDIO_OUT_B: now also U201.14 (S4B)
- net AUDIO_OUT_FILT: now also U201.15 (D4)
- net BYPASS_A: now also U201.2 (S1B), U201.7 (S2A)
- net BYPASS_B: now also U201.12 (S3B), U201.16 (S4A)
- net GND: now also J308.SH1, J308.SH2, C18.2, C18.2, U201.4 (GND); no longer J308.MP (MountPin)
- net SW_IN1: now also U201.19 (IN1)
- net SW_IN2: now also U201.8 (IN2)
- net SW_IN3: now also U201.9 (IN3)
- net SW_IN4: now also U201.17 (IN4)
- new net ~{SW_EN}: U201.18 (~{EN})
Other:
- note added: "OUTPUT FILTER PASSBAND: 20Hz - 25kHz"
- note added: "PLACE C201 AS CLOSE TO J201 AS POSSIBLE PLACE C210 AS CLOSE TO J203 AS POSSIBLE CAPACITORS C201, C202, C209, C210: 10% TOLERANCE, C0G/NP0 Dielectric PLACE CHASSIS GROUNDS AS CLOSE TO AUDIO JACKS AS POSSIBLE PLACE BYPASS CAPACITORS AS CLOSE TO ICS OR CONNECTORS AS POSSIBLE PLACE CONNECTORS NEAR BOARD EDGE PLACE AUDIO COMPONENTS NEAR EACH OTHER AND AWAY FROM OTHER CIRCUITS"
- note removed: "PLACE C201 AS CLOSE TO J201 AS POSSIBLE PLACE C210 AS CLOSE TO J203 AS POSSIBLE CAPACITORS C201, C202, C209, C210: 10% TOLERANCE, METALLIZED PET FILM DIELECTRIC PLACE CHASSIS GROUNDS AS CLOSE TO AUDIO JACKS AS POSSIBLE PLACE BYPASS CAPACITORS AS CLOSE TO ICS OR CONNECTORS AS POSSIBLE PLACE CONNECTORS NEAR BOARD EDGE PLACE AUDIO COMPONENTS NEAR EACH OTHER AND AWAY FROM OTHER CIRCUITS"
- company: ALESSANDRO RIZZONI -> Alessandro Rizzoni
- title: BASEBOARD -> Baseboard
