File: hardware/cad/audio.kicad_sch (KiCad schematic)
At the start: 18 parts, among them J201 ACJS-IHS, J203 ACJS-IHS, J308 SFV20R-2STE1HLF, U201 ADG5434

Commit message: started documentation
Parts:
- renumbered C414 to C202, C18 to C203, C18 to C204, C38 to C205, C418 to C206, C38 to C207, C418 to C208, C414 to C209, G2 to G201, G2 to G202, J308 to J202
Other:
- note removed: "Effects Board"

Commit message: minor changes before moving to new power supply topology
Connections:
- net AUDIO_IN_A: now also U201.20 (S1A); no longer U201.1 (D1)
- net AUDIO_IN_FILT: now also U201.1 (D1); no longer U201.20 (S1A)

Commit message: cleanup
Parts:
- removed C205: 100nF, Capacitor_SMD:C_0402_1005Metric, symbol Device:C
- removed C206: 2.2μF, Capacitor_SMD:C_0603_1608Metric, symbol Device:C
- removed J202: SFV20R-2STE1HLF, Library:AMPHENOL_SFV20R-2STE1HLF, symbol Library:Conn_01x20_SHIELD
- added C209: 100nF, Capacitor_SMD:C_0402_1005Metric, symbol Device:C
- added C210: 2.2μF, Capacitor_SMD:C_0603_1608Metric, symbol Device:C
- added J203: SFV20R-2STE1HLF, Library:AMPHENOL_SFV20R-2STE1HLF, symbol Library:Conn_01x20_SHIELD
- renumbered C210 to C202, C202 to C203, C209 to C204, C203 to C205, C204 to C206, J203 to J202
Connections:
- net +9V: now also C207.2, C208.2, J203.8 (Pin_8), J203.9 (Pin_9)
- net -9V: now also C209.2, C210.2, J203.12 (Pin_12), J203.13 (Pin_13); no longer C207.2, C208.2
- net AUDIO_IN_A: now also J203.2 (Pin_2)
- net AUDIO_IN_B: now also J203.17 (Pin_17)
- net AUDIO_OUT_A: now also J203.4 (Pin_4)
- net AUDIO_OUT_B: now also J203.19 (Pin_19)
- net GND: now also C209.1, C210.1, J203.1 (Pin_1), J203.10 (Pin_10), J203.11 (Pin_11), J203.14 (Pin_14), J203.15 (Pin_15), J203.16 (Pin_16), J203.18 (Pin_18), J203.20 (Pin_20), J203.3 (Pin_3), J203.5 (Pin_5), J203.6 (Pin_6), J203.7 (Pin_7), J203.SH1, J203.SH2
- net AUDIO_IN- renamed AUDIO_IN
Other:
- note removed: "AUDIO INPUT"
- note removed: "AUDIO OUTPUT"
- note removed: "EFFECT BOARD INTERFACE"
- note removed: "SWITCHING"
- moved on the sheet: C201, C202, C203, C204, C205, C206, J201, J202, R201, R202, U201
