File: hardware/cad/baseboard.kicad_pcb (KiCad board)
At the start: 6 copper layers, 100 x 60 mm, 109 parts, among them J201 1/4" JACK, STEREO, J202 FFC CONNECTOR, J203 1/4" JACK, STEREO, J301 JACK, DC, J401 6-440054-2, J403 2x2 PIN HEADER, J404 6-440054-2, J406 6-440054-2, J408 6-440054-2, Q401 DMN2050, Q402 DMN2050, U201 ADG5434, U301 LM337, U302 LM317, U303 ADP5070, U304 LM317, U401 STM32G031K8U6

Commit message: an inappropriately large commit
Parts:
- removed FID201: FIDUCIAL, Fiducial:Fiducial_0.5mm_Mask1mm
- removed G101: OSHW LOGO, Symbol:OSHW-Logo_7.5x8mm_SilkScreen
- removed G102: ESD SYMBOL, Symbol:ESD-Logo_8.9x8mm_SilkScreen
- added G***: LOGO, LOGO, F.Cu at (269.0, 112.9)
- added H401: JLC_TOOLING_HOLE, Library:JLC_Tooling_hole, F.Cu at (269.7, 106.7)
- added H402: JLC_TOOLING_HOLE, Library:JLC_Tooling_hole, F.Cu at (173.7, 106.7)
- added H403: JLC_TOOLING_HOLE, Library:JLC_Tooling_hole, F.Cu at (173.7, 160.7)
- added H404: JLC_TOOLING_HOLE, Library:JLC_Tooling_hole, F.Cu at (269.7, 160.7)
- C202, C209, C308: footprint Capacitor_SMD:C_0603_1608Metric -> Capacitor_SMD:C_0805_2012Metric
- D401: value TVS -> RSB12JS2
- J201, J203: value 1/4" JACK, STEREO -> ACJS-IHS
- J202: value FFC CONNECTOR -> SFV20R-2STE1HLF
- J301: value JACK, DC -> PJ-063AH
- TP301: value TEST POINT -> DC_IN; footprint TestPoint:TestPoint_Pad_D1.0mm -> Library:TestPoint_Pad_D1.0mm
- TP302: value TEST POINT -> GND; footprint TestPoint:TestPoint_Pad_D1.0mm -> Library:TestPoint_Pad_D1.0mm
- TP303: value TEST POINT -> -9V; footprint TestPoint:TestPoint_Pad_D1.0mm -> Library:TestPoint_Pad_D1.0mm
- TP304: value TEST POINT -> +9V; footprint TestPoint:TestPoint_Pad_D1.0mm -> Library:TestPoint_Pad_D1.0mm
- TP305: value TEST POINT -> +3V3; footprint TestPoint:TestPoint_Pad_D1.0mm -> Library:TestPoint_Pad_D1.0mm
- U201, U303: footprint Library:LFCSP-20-1EP_4x4mm_P0.5mm_EP2.6x2.6mm_ThermalVias -> Library:LFCSP-20-1EP_4x4mm_P0.5mm_EP2.6x2.6mm
- U301: value LM337 -> LM337KVURG3; footprint Library:TO-252-2_THERMAL_PAD -> Library:TO-252-2
- U302, U304: value LM317 -> LM317MDT-TR; footprint Library:TO-252-2_THERMAL_PAD -> Library:TO-252-2
- U401: footprint Library:QFN-32-1EP_5x5mm_P0.5mm_EP3.45x3.45mm_ThermalVias -> Library:QFN-32-1EP_5x5mm_P0.5mm_EP3.45x3.45mm
- moved J403 148.0 mm to (230.6, 141.1), turned to 180 degrees
- moved D401 144.6 mm to (230.6, 137.1), turned to -90 degrees
- moved C205 143.5 mm to (195.2, 157.3)
- moved C206 143.5 mm to (195.1, 156.0)
- moved C208 143.5 mm to (198.3, 156.0)
- moved J202 143.5 mm to (196.7, 161.2)
- moved C207 143.5 mm to (198.2, 157.3)
- moved C204 139.5 mm to (193.6, 139.9)
- moved U201 139.3 mm to (196.7, 139.7)
- moved C203 139.0 mm to (200.1, 140.2), turned to -90 degrees
- moved L301 138.2 mm to (260.7, 132.4)
- moved C314 138.2 mm to (265.6, 136.0)
- moved C302 137.9 mm to (265.1, 119.2)
- moved C306 137.9 mm to (265.8, 149.3)
- moved C313 137.9 mm to (246.4, 135.5)
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Connections:
- C203 pad 1: GND -> +9V
- C203 pad 2: +9V -> GND
- J202 pad SH1: (no net) -> GND
- J202 pad SH2: (no net) -> GND
- J301 pad S1: (no net) -> GND
- J301 pad S2: (no net) -> GND
- NT301 pad 1: GND -> GND1
- NT301 pad 2: GND1 -> GND
- U201 pad 1: AUDIO_IN_FILT -> AUDIO_IN_A
- U201 pad 18: SW_EN -> ~{SW_EN}
- U201 pad 20: AUDIO_IN_A -> AUDIO_IN_FILT
- U401 pad 1: unconnected-(U401-PB9-Pad1) -> FTSW_B
- U401 pad 10: SW_IN2 -> LEDA_EN
- U401 pad 11: SW_IN3 -> unconnected-(U401-PA4-Pad11)
- U401 pad 17: unconnected-(U401-PB2-Pad17) -> SW_IN1
- U401 pad 18: unconnected-(U401-PA8-Pad18) -> ~{SW_EN}
- U401 pad 19: unconnected-(U401-PA9/NC-Pad19) -> SW_IN4
- U401 pad 2: unconnected-(U401-PC14-Pad2) -> LEDB_EN
- U401 pad 20: unconnected-(U401-PC6-Pad20) -> SW_IN3
- U401 pad 21: -9V_EN -> SW_IN2
- U401 pad 22: +9V_EN -> unconnected-(U401-PA11/PA9-Pad22)
- U401 pad 28: FTSW_B -> unconnected-(U401-PB4-Pad28)
- U401 pad 29: LEDB_EN -> unconnected-(U401-PB5-Pad29)
- U401 pad 31: FTSW_A -> -9V_EN
- U401 pad 32: LEDA_EN -> +9V_EN
- U401 pad 7: SW_EN -> unconnected-(U401-PA0-Pad7)
- U401 pad 8: SW_IN4 -> unconnected-(U401-PA1-Pad8)
- U401 pad 9: SW_IN1 -> FTSW_A
Routing:
- net SW_EN: track 48.3 -> 0.00 mm, vias 3 -> 0
- net ~{SW_EN}: track 0.00 -> 37.7 mm, vias 0 -> 2
- net +3V3: track 39.8 -> 62.2 mm, vias 10 -> 13
- net /MICROCONTROLLER/SWDCK: track 26.7 -> 14.3 mm, vias 2 -> 0
- net AUDIO_OUT_B: track 12.5 -> 23.8 mm
- net AUDIO_OUT_A: track 7.72 -> 18.6 mm
- net AUDIO_IN_A: track 15.2 -> 25.8 mm, vias 2 -> 0
- net /MICROCONTROLLER/SWDIO: track 29.9 -> 19.4 mm, vias 2 -> 0
- net SW_IN3: track 49.9 -> 39.5 mm, vias 3 -> 2
- net SW_IN4: track 46.9 -> 36.5 mm, vias 3 -> 2
- net AUDIO_IN_B: track 8.15 -> 18.3 mm
- net +9V_EN: track 17.0 -> 26.7 mm
- net -9V_EN: track 15.7 -> 25.3 mm
- net /AUDIO/AUDIO_IN-: track 9.03 -> 18.0 mm
- net /AUDIO/AUDIO_OUT: track 9.05 -> 18.0 mm
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- added copper zone on F.Cu, net GND
- added copper zone on In2.Cu, net GND
Other:
- board size 100 x 60 mm -> 102.3 x 60 mm
- board text added: "#D2960FFF"
- board text added: "0"
- board text added: "0 mm"
- board text added: "0.01 mm"
- board text added: "0.0152 mm"
- board text added: "0.02"
- board text added: "0.035 mm"
- board text added: "0.0900 mm / 0.0900 mm"
- board text added: "0.1 mm"
- board text added: "0.2500 mm"
- board text added: "0.5548 mm"
- board text added: "1"
- board text added: "1.6000 mm"
- board text added: "102.3000 mm x 60.0000 mm"
- board text added: "1: MANUFACTURE TO IPC CLASS 2"
- board text added: "2023-08 Rev. A - AIR"
- board text added: "3.3"
- board text added: "3V3"
- board text added: "4.5"
- board text added: "6"
- board text added: "9VDC"
- board text added: "B.Cu (Ground)"
- board text added: "B.Mask"
- board text added: "B.Paste"
- board text added: "B.Silkscreen"
- board text added: "BOARD CHARACTERISTICS"
- board text added: "Baseboard V1.0"
- board text added: "Board Thickness:"
- board text added: "Board overall dimensions:"
- board text added: "Bottom Silk Screen"
- board text added: "Bottom Solder Mask"
- board text added: "Bottom Solder Paste"
- board text added: "CK"
- board text added: "Castellated pads:"
- board text added: "Color"
- board text added: "Copper"
- board text added: "Copper Finish:"
- board text added: "Copper Layer Count:"
- board text added: "Dielectric"
- board text added: "EFFECTS INTERFACE"
- board text added: "ENIG"
- board text added: "Edge card connectors:"
- board text added: "Epsilon R"
- board text added: "F.Cu (Signal)"
- board text added: "F.Mask"
- board text added: "F.Paste"
- board text added: "F.Silkscreen"
- board text added: "FR4"
- board text added: "GND"
- board text added: "Green"
- board text added: "INITIAL RELEASE"
- board text added: "IO"
- board text added: "Impedance Control:"
- board text added: "In1.Cu (Ground)"
- board text added: "In2.Cu (Signal)"
- board text added: "In3.Cu (Ground)"
- board text added: "In4.Cu (Power)"
- board text added: "Layer Name"
- board text added: "Loss Tangent"
- board text added: "Material"
- board text added: "Min hole diameter:"
- board text added: "Min track/spacing:"
- board text added: "No"
- board text added: "Not specified"
- board text added: "Plated Board Edge:"
- board text added: "SWD"
- board text added: "Thickness (mm)"
- board text added: "Top Silk Screen"
- board text added: "Top Solder Mask"
- board text added: "Top Solder Paste"
- board text added: "Type"
- board text added: "White"
- board text added: "copper"
- board text added: "core"
- board text added: "prepreg"
- board text removed: "Baseboard V1.0 AIR:2023-07-30"
