File: hardware/cad/power.kicad_sch (KiCad schematic)
At the start: 53 parts, among them J301 PJ-063AH, U301 LM337KVURG3, U302 LM317MDT-TR, U303 ADP5070, U304 LM317MDT-TR

Commit message: started documentation
Parts:
- removed C201: 150pF, Capacitor_SMD:C_0805_2012Metric, symbol Device:C
- removed C318: 10μF, Capacitor_SMD:C_1210_3225Metric, symbol Device:C
- removed D203: DFLZ13Q-7, Library:D_PowerDI-123_THERMAL_PAD, symbol Library:DFLZ13Q-7
- removed D304: DFLS240L-7, Library:D_PowerDI-123_THERMAL_PAD, symbol Library:RSX051VAM30TR
- removed TP203: GND, TestPoint:TestPoint_Pad_D1.0mm, symbol Connector:TestPoint
- removed TP204: DC_IN, TestPoint:TestPoint_Pad_D1.0mm, symbol Connector:TestPoint
- removed TP305: +3V3, TestPoint:TestPoint_Pad_D1.0mm, symbol Connector:TestPoint
- removed U304: LM317MDT-TR, Library:TO-252-2, symbol Regulator_Linear:LM317_TO-252
- added C302: 3.3n, symbol Device:C
- added C321: 22u, symbol Device:C
- added L304: 2.2u, symbol Device:L
- added R314: 470k, symbol Device:R_US
- added R315: 11k, symbol Device:R_US
- added R316, R318, R319: 47k, symbol Device:R_US
- added R317: 549, symbol Device:R_US
- added R320: 5.6k, symbol Device:R_US
- added R321: 100k, symbol Device:R_US
- added TP301: DC_IN, TestPoint:TestPoint_Pad_D1.0mm, symbol Connector:TestPoint
- added TP302: GND, TestPoint:TestPoint_Pad_D1.0mm, symbol Connector:TestPoint
- added U305: TPS259474L, symbol Library:TI_TPS25947
- added U306: TPS62170DSG, Package_SON:WSON-8-1EP_2x2mm_P0.5mm_EP0.9x1.6mm_ThermalVias, symbol Regulator_Switching:TPS62170DSG
- C305: value 10μF -> 2.2n; footprint Capacitor_SMD:C_1210_3225Metric -> (none); Manufacturer Murata -> (none); Part Number GRM32EC72A106KE05L -> (none)
- C313: value 10μF -> 22u; footprint Capacitor_SMD:C_1210_3225Metric -> (none); Manufacturer Murata -> (none); Part Number GRM32EC72A106KE05L -> (none)
- C316: value 2.2μF -> 22u; footprint Capacitor_SMD:C_0603_1608Metric -> (none); Manufacturer Murata -> (none); Part Number GRM188Z71E225KE43D -> (none)
- R308: value 200Ω -> 470k; footprint Resistor_SMD:R_0402_1005Metric -> (none); Manufacturer KOA Speer Electronics -> (none); Part Number RK73H1ETTP2000F -> (none)
- R311: value 120Ω -> 150k; footprint Resistor_SMD:R_0402_1005Metric -> (none); Manufacturer KOA Speer Electronics -> (none); Part Number RK73H1ETTP1200F -> (none)
- renumbered FID302 to FID301, CHS201 to G301
Connections:
- net +3V3: now also C313.1, R308.1, L304.2, R319.1, R321.1, U306.6 (VOS); no longer R311.1
- net DC_IN: now also C316.1, C321.1, R318.1, TP301.1, U305.6 (OUT), U306.2 (VIN), U306.3 (EN); no longer C305.2, C313.2
- net DC_IN_RAW: now also R314.1, U305.5 (IN)
- net GND: now also C305.2, C313.2, C316.2, C302.2, C321.2, R316.2, R317.2, R320.1, TP302.1, U305.8 (GND); no longer C305.1, C313.1, C316.1, R308.2
- removed net 3V3REG_FB: C316.2, R308.1, R311.2
- new net: R314.2, R315.1, U305.1 (EN/UVLO)
- new net: R317.1, U305.9 (ILM)
- new net: R315.2, R316.1, U305.2 (OVLO)
- new net: C305.1, U305.10 (ITIMER)
- new net: R318.2, R320.2, U305.4 (~{FLT}/PGTH)
- new net: C302.1, U305.7 (DVDT)
- new net: R308.2, R311.1, U306.5 (FB)
- new net: L304.1, U306.7 (SW)
- new net: R311.2, U306.1 (PGND), U306.4 (AGND), U306.9 (PAD)
- new net DC_IN_PG: R319.2, U305.3 (AUXOFF/PG)
- new net PG_3v3: R321.2, U306.8 (PG)
Other:
- note added: "+12VDC CENTER NEGATIVE"
- note removed: "+9-12VDC CENTER NEGATIVE"
- moved on the sheet: J301

Commit message: minor changes before moving to new power supply topology
Parts:
- removed D302, D303: DFLS240L-7, Library:D_PowerDI-123_THERMAL_PAD, symbol Library:RSX051VAM30TR
- removed FID301: FIDUCIAL, Fiducial:Fiducial_0.5mm_Mask1mm, symbol Mechanical:Fiducial
- removed L301, L302: 22μH, Library:L_TDK_VLS6045EX_VLS6045AF, symbol Device:L
- removed L304: 2.2u, symbol Device:L
- removed NT301: NET TIE, Library:Net_Tie, symbol Device:NetTie_2
- removed U301: LM337KVURG3, Library:TO-252-2, symbol Regulator_Linear:LM337_TO252
- removed U302: LM317MDT-TR, Library:TO-252-2, symbol Regulator_Linear:LM317_TO-252
- removed U303: ADP5070, Library:LFCSP-20-1EP_4x4mm_P0.5mm_EP2.6x2.6mm, symbol Library:ADP5070ACPZ
- removed U305: TPS259474L, symbol Library:TI_TPS25947
- added C318, C322: 10μF, Capacitor_SMD:C_1210_3225Metric, symbol Device:C
- added C323, C324: C, symbol Device:C
- added D301, D302: D_Schottky_Filled, symbol Device:D_Schottky_Filled
- added J302: USB_C_Receptacle_USB2.0_14P, symbol Connector:USB_C_Receptacle_USB2.0_14P
- added L301, L302: L, symbol Library:L_Coupled_POLAR
- added Q301, Q302: Q_NMOS_DSG, symbol Device:Q_NMOS_DSG
- added R322: 120Ω, Resistor_SMD:R_0402_1005Metric, symbol Device:R_US
- added R323, R324: 0R, symbol Device:R_US
- added R325, R327, R328: R_US, symbol Device:R_US
- added U301: DS1086L, Package_SO:TSSOP-8_3x3mm_P0.65mm, symbol Library:ANALOG_MAXIM_DS1086L
- added U302: TPS259474L, symbol Library:TI_TPS25947
- added U303: 74LVC1GU04DRL, Package_TO_SOT_SMD:SOT-553, symbol 74xGxx:74LVC1GU04DRL
- added U304, U305: LT3580xDD, Package_DFN_QFN:DFN-8-1EP_3x3mm_P0.5mm_EP1.66x2.38mm, symbol Regulator_Switching:LT3580xDD
- added U307: LM337KVURG3, Library:TO-252-2, symbol Regulator_Linear:LM337_TO252
- added U308: LM317MDT-TR, Library:TO-252-2, symbol Regulator_Linear:LM317_TO-252
- added U309, U310: LM74700, Package_TO_SOT_SMD:SOT-23-6, symbol Power_Management:LM74700
- added U312: TUSB320, Package_DFN_QFN:Texas_X2QFN-12_1.6x1.6mm_P0.4mm, symbol Interface_USB:TUSB320
- C301, C306, C311, C314, C315: value 10μF -> C; footprint Capacitor_SMD:C_1210_3225Metric -> (none); Manufacturer Murata -> (none); Part Number GRM32EC72A106KE05L -> (none)
- C302: value 3.3n -> 2.2n
- C303: value 2.2μF -> 3.3n; footprint Capacitor_SMD:C_0603_1608Metric -> (none); Manufacturer Murata -> (none); Part Number GRM188Z71E225KE43D -> (none)
- C304, C307: value 10μF -> 22u; footprint Capacitor_SMD:C_1210_3225Metric -> (none); Manufacturer Murata -> (none); Part Number GRM32EC72A106KE05L -> (none)
- C305: value 2.2n -> C
- C308: value 58nF -> C; footprint Capacitor_SMD:C_0805_2012Metric -> (none); Manufacturer Kemet -> (none); Part Number C0805C564K5RAC7800 -> (none)
- C309, C312: value 2.2μF -> C; footprint Capacitor_SMD:C_0603_1608Metric -> (none); Manufacturer Murata -> (none); Part Number GRM188Z71E225KE43D -> (none)
- C310: value 10nF -> C; footprint Capacitor_SMD:C_0603_1608Metric -> (none); Manufacturer TDK -> (none); Part Number CGA3E2X7R1H103K080AA -> (none)
- C313: value 22u -> C
- C319, C320: value 10μF -> 2.2μF; footprint Capacitor_SMD:C_1210_3225Metric -> Capacitor_SMD:C_0603_1608Metric; Part Number GRM32EC72A106KE05L -> GRM188Z71E225KE43D
- C321: value 22u -> 10μF; footprint (none) -> Capacitor_SMD:C_1210_3225Metric; Manufacturer (none) -> Murata; Part Number (none) -> GRM32EC72A106KE05L
- L303: value 22μH -> 2.2u; footprint Library:L_TDK_VLS6045EX_VLS6045AF -> (none); Manufacturer Bourns -> (none); Part Number SRP5030WA-220M -> (none)
- R301: value 750Ω -> 470k; footprint Resistor_SMD:R_0402_1005Metric -> (none); Manufacturer KOA Speer Electronics -> (none); Part Number RK73H1ETTP7500F -> (none)
- R302: value 120Ω -> 11k; footprint Resistor_SMD:R_0402_1005Metric -> (none); Manufacturer KOA Speer Electronics -> (none); Part Number RK73H1ETTP1200F -> (none)
- R303: value 750Ω -> 47k; footprint Resistor_SMD:R_0402_1005Metric -> (none); Manufacturer KOA Speer Electronics -> (none); Part Number RK73H1ETTP7500F -> (none)
- R304: value 33kΩ -> 47k; footprint Resistor_SMD:R_0402_1005Metric -> (none); Manufacturer KOA Speer Electronics -> (none); Part Number RK73H1ETTP3302F -> (none)
- R305: value 120Ω -> 5.6k; footprint Resistor_SMD:R_0402_1005Metric -> (none); Manufacturer KOA Speer Electronics -> (none); Part Number RK73H1ETTP1200F -> (none)
- R306: value 3.3kΩ -> 47k; footprint Resistor_SMD:R_0402_1005Metric -> (none); Manufacturer KOA Speer Electronics -> (none); Part Number RK73H1ETTP3301F -> (none)
- R307: value 71.5kΩ -> 549; footprint Resistor_SMD:R_0402_1005Metric -> (none); Manufacturer KOA Speer Electronics -> (none); Part Number RK73H1ETTP7152F -> (none)
- R308: value 470k -> R_US
- R309: value 62.5kΩ -> R_US; footprint Resistor_SMD:R_0402_1005Metric -> (none); Manufacturer KOA Speer Electronics -> (none); Part Number RK73H1ETTP6252F -> (none)
- R310: value 1MΩ -> R_US; footprint Resistor_SMD:R_0402_1005Metric -> (none); Manufacturer KOA Speer Electronics -> (none); Part Number RK73H1ETTP1004F -> (none)
- R311: value 150k -> R_US
- R312: value 1MΩ -> 100k; footprint Resistor_SMD:R_0402_1005Metric -> (none); Manufacturer KOA Speer Electronics -> (none); Part Number RK73H1ETTP1004F -> (none)
- R313: value 71.5kΩ -> 0R; footprint Resistor_SMD:R_0402_1005Metric -> (none); Manufacturer KOA Speer Electronics -> (none); Part Number RK73H1ETTP7152F -> (none); now not fitted
- R314: value 470k -> 0R; now not fitted
- R315: value 11k -> 470k
- R316: value 47k -> 150k
- R317: value 549 -> R_US
- R318: value 47k -> R_US
- R319: value 47k -> 750Ω; footprint (none) -> Resistor_SMD:R_0402_1005Metric; Manufacturer (none) -> KOA Speer Electronics; Part Number (none) -> RK73H1ETTP7500F
- R320: value 5.6k -> 750Ω; footprint (none) -> Resistor_SMD:R_0402_1005Metric; Manufacturer (none) -> KOA Speer Electronics; Part Number (none) -> RK73H1ETTP7500F
- R321: value 100k -> 120Ω; footprint (none) -> Resistor_SMD:R_0402_1005Metric; Manufacturer (none) -> KOA Speer Electronics; Part Number (none) -> RK73H1ETTP1200F
- TP301: value DC_IN -> GND
- TP302: value GND -> DC_IN
Connections:
- net VSW1A is gone; now on net GND: C314.2
- net VSW_COMP2 is gone; now on net DC_IN_PG: R306.2
- net VSW_SOFT_START is gone; now on net GND: R307.2
- net +12V_RAW: now also C315.1, R318.1, C318.2, D302.1 (K), U308.3 (VI); no longer C306.2, C319.2, C320.2, R312.2
- net +3V3: now also C316.1, L303.2, R306.1, R312.1, R315.1, U312.12 (VDD); no longer C313.1, R308.1, R319.1, R321.1
- net +9V: now also C322.2, R322.1, U308.2 (VO); no longer C311.2, R305.1
- net +9VREG_FBP: now also C320.2, R320.1, R322.2, U308.1 (ADJ); no longer C309.2, R303.1, R305.2
- net +9V_EN: now also U305.5 (~{SHDN})
- net -12V_RAW: now also C314.1, R317.1, L301.4, U307.2 (VI); no longer C301.2, C315.2, R310.1
- net -9V: now also C321.2, R321.1, U307.3 (VO); no longer C304.2, R302.1
- net -9VREG_FBN: now also C319.2, R319.1, R321.2, U307.1 (ADJ); no longer C303.2, R301.1, R302.2
- net -9V_EN: now also U304.5 (~{SHDN})
- net DC_IN: now also C304.1, C308.1, C309.1, R304.1, TP302.1, C324.1, L301.2, L302.2, Q302.2 (S), R328.2, U302.6 (OUT), U304.3 (VIN), U305.3 (VIN), U310.6 (ANODE); no longer C307.2, C316.1, C321.1, R318.1, TP301.1, U306.2 (VIN), U306.3 (EN)
- net DC_IN_PG: now also U302.3 (AUXOFF/PG); no longer R319.2
- net DC_IN_RAW: now also R301.1, U302.5 (IN); no longer R314.1
- net GND: now also C301.2, C303.2, C304.2, C306.2, C307.2, C308.2, C309.2, C310.2, C311.2, C315.2, C317.1, C319.1, C320.1, C321.1, R305.1, R310.1, R311.1, R313.2, R314.2, R319.2, R320.2, TP301.1, U306.1 (PGND), U306.4 (AGND), U306.9 (PAD), C318.1, C322.1, D301.1 (K), J302.A1 (GND), J302.A12 (GND), J302.B1 (GND), J302.B12 (GND), J302.S1 (SHIELD), L302.4, U301.4 (GND), U302.8 (GND), U303.3 (GND), U304.9 (GND), U305.9 (GND), U309.2 (GND), U310.2 (GND), U312.10 (GND), U312.3 (PORT), U312.5 (ADDR); no longer C301.1, C303.1, C304.1, C306.1, C308.1, C309.1, C310.1, C311.1, C312.1, C313.2, C321.2, R301.2, R307.1, R313.1, R317.2, R320.1, TP302.1
- net PG_3v3: now also R312.2; no longer R321.2
- net at R315.2, R316.1: now also U306.5 (FB)
- net at C305.1: now also R308.1
- net at R318.2: now also U305.1 (FB); no longer R320.2
- net at C302.1: now also U302.10 (ITIMER)
- net at U306.7 (SW): now also L303.1
- removed net GND1: C307.1, C315.1, C317.1, C319.1, C320.1, L303.1
- removed net VSW1B: C314.1, L303.2
- net VSW_COMP1: no longer names the net of R304.2
- net VSW_COMP1: now also R305.2, U302.4 (~{FLT}/PGTH)
- removed net VSW_FB1: R312.1, R313.2
- net VSW_FB2: no longer names the net of R310.2
- net VSW_FB2: now also U304.6 (RT); no longer R309.1
- net VSW_VREF: no longer names the net of R309.2
- net VSW_VREF: now also U305.2 (VC)
- net VSW_VREG: no longer names the net of C312.2
- net VSW_VREG: now also D301.2 (A), L301.3
- new net: R328.1, U310.3 (EN)
- new net: R317.2, U304.1 (FB)
- new net: R308.2, U304.2 (VC)
- new net: C312.1, L301.1, U304.4 (SW)
- new net: C310.1, U304.7 (SS)
- new net: R313.1, R323.1, U304.8 (SYNC)
- new net: R301.2, R302.1, U302.1 (EN/UVLO)
- new net: C324.2, U310.1 (VCAP)
- new net: C307.1, Q301.1 (D), Q302.1 (D), U306.2 (VIN), U306.3 (EN), U309.4 (CATHODE), U310.4 (CATHODE)
- new net: Q302.3 (G), U310.5 (GATE)
- new net: J302.A5 (CC1), U312.1 (CC1)
- new net: J302.B5 (CC2), U312.2 (CC2)
- new net: R325.2, U312.4 (VBUS_DET)
- new net: C313.2, D302.2 (A), L302.3
- new net: R314.1, R324.1, U305.8 (SYNC)
- new net: R302.2, R303.1, U302.2 (OVLO)
- new net: C306.1, R309.1
- new net: C323.1, J302.A4 (VBUS), J302.A9 (VBUS), J302.B4 (VBUS), J302.B9 (VBUS), Q301.2 (S), R325.1, R327.2, U309.6 (ANODE)
- new net: Q301.3 (G), U309.5 (GATE)
- new net: C303.1, U302.7 (DVDT)
- new net: R307.1, U302.9 (ILM)
- new net: C323.2, U309.1 (VCAP)
- new net: R327.1, U309.3 (EN)
- new net: R311.2, U305.6 (RT)
- new net: C313.1, L302.1, U305.4 (SW)
- new net: C311.1, U305.7 (SS)
- new net +12V_SYNC: R324.2, U301.1 (OUT), U303.2
- new net +3.3V: C301.1, U301.3 (VCC), U303.5 (VCC)
- new net -12V_SYNC: R323.2, U303.4
- new net uC_USB_DM: J302.A6 (D+), J302.B6 (D+)
- new net uC_USB_DP: J302.A7 (D-), J302.B7 (D-)
- no-connect marks 1 -> 0
Other:
- note added: "Minimize loop areas"
- note removed: "+3.3V LINEAR REGULATOR"
- note removed: "+9V LINEAR REGULATOR"
- note removed: "-9V LINEAR REGULATOR"
- note removed: "POWER INPUT"
- note removed: "SOFT START RESISTOR R407 = 71.5kΩ t_SS = 29ms"
- note removed: "±12V 200mA SWITCHING REGULATOR"

Commit message: started modeling circuits
Parts:
- added U311: PI3USB221E, symbol Library:DIODES_PI3USB221E

Commit message: cleanup
Parts:
- removed C308, C309: C, symbol Device:C
- removed C316: 22u, symbol Device:C
- removed R308, R309, R310: R_US, symbol Device:R_US
- removed R324: 0R, symbol Device:R_US
- removed U301: DS1086L, Package_SO:TSSOP-8_3x3mm_P0.65mm, symbol Library:ANALOG_MAXIM_DS1086L
- removed U303: 74LVC1GU04DRL, Package_TO_SOT_SMD:SOT-553, symbol 74xGxx:74LVC1GU04DRL
- removed U304, U305: LT3580xDD, Package_DFN_QFN:DFN-8-1EP_3x3mm_P0.5mm_EP1.66x2.38mm, symbol Regulator_Switching:LT3580xDD
- removed U306: TPS62170DSG, Package_SON:WSON-8-1EP_2x2mm_P0.5mm_EP0.9x1.6mm_ThermalVias, symbol Regulator_Switching:TPS62170DSG
- added C307, C317, C318: C, symbol Device:C
- added C321: 22u, symbol Device:C
- added R319: R_US, symbol Device:R_US
- added R322: 470k, symbol Device:R_US
- added U306, U307: LT3580xDD, Package_DFN_QFN:DFN-8-1EP_3x3mm_P0.5mm_EP1.66x2.38mm, symbol Regulator_Switching:LT3580xDD
- added U308: TPS62170DSG, Package_SON:WSON-8-1EP_2x2mm_P0.5mm_EP0.9x1.6mm_ThermalVias, symbol Regulator_Switching:TPS62170DSG
- C305: value C -> 100n
- R312: value 100k -> R_US
- R313, R314: value 0R -> R_US; now fitted
- R315: value 470k -> 0R
- R316: value 150k -> 0R
- R317: value R_US -> 100k
- R323: value 0R -> 150k
- TP303: value -9V -> -12V
- TP304: value +9V -> +12V
- renumbered C324 to C308, C323 to C309, C307 to C316, C317 to C319, C318 to C320, C319 to C322, C320 to C323, C321 to C324, C322 to C325, J302 to J301, J301 to J302, Q302 to Q301, Q301 to Q302, R325 to R306, R306 to R307, R307 to R308, R328 to R309, R327 to R310, R319 to R320, R320 to R321, R321 to R324, R322 to R325, U311 to U301, U312 to U303, U310 to U304, U309 to U305, U307 to U309, U308 to U310
Connections:
- net +3.3V is gone; now on net +3V3: C301.1
- net -12V_SYNC is gone; now on net GND: R323.2
- net +3V3: now also R317.1, U301.10 (VDD), C321.1, R322.1, U308.6 (VOS); no longer R312.1, R315.1
- net +9V_EN: now also U307.5 (~{SHDN})
- net -9V_EN: now also U306.5 (~{SHDN})
- net DC_IN: now also C310.1, C311.1, U306.3 (VIN), U307.3 (VIN)
- net GND: now also C312.2, C313.2, R313.1, R314.1, R315.2, U301.5 (GND), C307.2, C317.2, C318.2, C321.2, U306.9 (GND), U307.9 (GND), U308.1 (PGND), U308.4 (AGND), U308.5 (FB), U308.9 (PAD); no longer C305.2, C314.2, C315.2, R311.1, R313.2, R314.2
- net PG_3v3: now also R317.2, U308.8 (PG); no longer R312.2
- net uC_USB_DM: now also U301.7 (D-); no longer J301.A6 (D+), J301.B6 (D+)
- net uC_USB_DP: now also U301.8 (D+); no longer J301.A7 (D-), J301.B7 (D-)
- net at R318.2: now also U306.1 (FB)
- net at D301.2 (A), L301.3: now also C314.2; no longer C312.2
- net at R316.1: now also U307.8 (SYNC); no longer R315.2
- net at L301.1: now also C314.1, U306.4 (SW); no longer C312.1
- net at R323.1: now also R322.2; no longer R313.1
- net at L303.1: now also U308.7 (SW)
- net at C316.1, Q301.1 (D), Q302.1 (D)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: now also U308.2 (VIN), U308.3 (EN)
- net at D302.2 (A), L302.3: now also C315.2; no longer C313.2
- net at C306.1: now also R311.1
- net at R311.2: now also U306.2 (VC)
- net at U301.1 (1D+): now also J301.A6 (D+)
- net at U301.2 (1D-): now also J301.A7 (D-)
- net at U301.3 (2D+): now also J301.B6 (D+)
- net at U301.4 (2D-): now also J301.B7 (D-)
- net at L302.1: now also C315.1, U307.4 (SW); no longer C313.1
- net +12V_RAW renamed +15V_RAW
- net +15V_RAW: now also C318.1, R319.1; no longer C315.1, R318.1
- net +9V renamed +12V
- net -12V_RAW renamed -15V_RAW
- net -15V_RAW: now also R318.1, C317.1; no longer C314.1, R317.1
- net -9V renamed -12V
- new net: R319.2, U307.1 (FB)
- new net: R312.2, U307.2 (VC)
- new net: R314.2, U307.6 (RT)
- new net: C313.1, U307.7 (SS)
- new net: R313.2, U306.6 (RT)
- new net: C312.1, U306.7 (SS)
- new net: R315.1, U306.8 (SYNC)
- new net: C307.1, R312.1
Other:
- note added: "+9-12V -> +/-15V -> +/-12V 12V sent to effects board for local linear regulation to +/-9V"
- note added: "+9-12VDC CENTER NEGATIVE"
- note removed: "+12VDC CENTER NEGATIVE"
- moved on the sheet: C309, C316, J301, Q302, R306, R310, U301, U303, U305
